Commit message: ajuste de parametros dinamicos

File: src/clase5/robot_description/dp/dp_params.xacro (robot description, xacro)
@@ -43,9 +43,9 @@
   <xacro:arg name="q1_min" default="-3.14" />                 <!-- límite físico inferior eje 1 -->
   <xacro:arg name="qp1_max" default="5.0" />                  <!-- límite físico velocidad eje 1 -->
-  <xacro:arg name="tau1_max" default="100.0" />               <!-- límite físico del esfuerzo aplicable en eje 1 -->
+  <xacro:arg name="tau1_max" default="1000.0" />               <!-- límite físico del esfuerzo aplicable en eje 1 -->
   <xacro:arg name="q2_max" default="3.14" />                  <!-- límite físico superior eje 2 -->
   <xacro:arg name="q2_min" default="-3.14" />                 <!-- límite físico inferior eje 2 -->
   <xacro:arg name="qp2_max" default="5.0" />                  <!-- límite físico velocidad eje 2 -->
-  <xacro:arg name="tau2_max" default="100.0" />               <!-- límite físico del esfuerzo aplicable en eje 2 -->
+  <xacro:arg name="tau2_max" default="1000.0" />               <!-- límite físico del esfuerzo aplicable en eje 2 -->
   <xacro:arg name="q1_ini" default="1.0" />                   <!-- condición inicial de posición -->
   <xacro:arg name="q2_ini" default="1.0" />                   <!-- condición inicial de posición -->

File: src/clase5/robot_description/mycobot_320_m5_2022/mycobot_320_m5_2022.xacro (robot description, xacro)
@@ -14,13 +14,22 @@
   <xacro:property name="link6_mass" value="0.0739" />
   <xacro:property name="flange_mass" value="0.035" />
-  <xacro:macro name="link_inertial" params="mass ixx iyy izz">
+  <xacro:macro name="link_inertial" params="xg yg zg mass ixx iyy izz">
     <inertial>
-      <origin xyz="0 0 0.0" rpy="0 0 0" />
+      <origin xyz="${xg} ${yg} ${zg}" rpy="0 0 0" />
       <mass value="${mass}" />
       <inertia ixx="${ixx}" ixy="0.0" ixz="0.0" iyy="${iyy}" iyz="0.0" izz="${izz}" />
     </inertial>
   </xacro:macro>
+  <!-- World link -->
+  <link name="world" />
+  <!-- Junta fija entre world y base_link -->
+  <joint name="fixed" type="fixed">
+    <parent link="world" />
+    <child link="base_link" />
+    <origin xyz="0 0 0" rpy="0 0 0" />
+  </joint>
   <link name="base_link">
-    <xacro:link_inertial mass="${base_mass}" ixx="0.000148" iyy="0.000148" izz="0.000096"/>
+    <xacro:link_inertial xg="0" yg="0" zg="0" mass="${base_mass}" ixx="0.000148" iyy="0.000148"
+      izz="0.000096" />
     <visual>
       <geometry>
@@ -37,5 +46,6 @@
   </link>
   <link name="link1">
-    <xacro:link_inertial mass="${link1_mass}" ixx="0.000148" iyy="0.000148" izz="0.000096"/>
+    <xacro:link_inertial xg="0" yg="0" zg="-0.078" mass="${link1_mass}" ixx="0.000148"
+      iyy="0.000148" izz="0.000096" />
     <visual>
       <geometry>
@@ -52,5 +62,6 @@
   </link>
   <link name="link2">
-    <xacro:link_inertial mass="${link2_mass}" ixx="0.000148" iyy="0.000148" izz="0.000096"/>
+    <xacro:link_inertial xg="0" yg="0" zg="-0.04" mass="${link2_mass}" ixx="0.000148" iyy="0.000148"
+      izz="0.000096" />
     <visual>
       <geometry>
@@ -67,5 +78,6 @@
   </link>
   <link name="link3">
-    <xacro:link_inertial mass="${link3_mass}" ixx="0.000148" iyy="0.000148" izz="0.000096"/>
+    <xacro:link_inertial xg="0" yg="0" zg="0.039" mass="${link3_mass}" ixx="0.000148" iyy="0.000148"
+      izz="0.000096" />
     <visual>
       <geometry>
@@ -82,5 +94,6 @@
   </link>
   <link name="link4">
-    <xacro:link_inertial mass="${link4_mass}" ixx="0.000103" iyy="0.000103" izz="0.000096"/>
+    <xacro:link_inertial xg="0" yg="0.0024" zg="-0.05" mass="${link4_mass}" ixx="0.000103"
+      iyy="0.000103" izz="0.000096" />
     <visual>
       <geometry>
@@ -97,5 +110,6 @@
   </link>
   <link name="link5">
-    <xacro:link_inertial mass="${link5_mass}" ixx="0.000103" iyy="0.000103" izz="0.000096"/>
+    <xacro:link_inertial xg="0" yg="0" zg="-0.05" mass="${link5_mass}" ixx="0.000103" iyy="0.000103"
+      izz="0.000096" />
     <visual>
       <geometry>
@@ -112,5 +126,6 @@
   </link>
   <link name="link6">
-    <xacro:link_inertial mass="${link6_mass}" ixx="0.00006649" iyy="0.00006649" izz="0.000096"/>
+    <xacro:link_inertial xg="0" yg="0" zg="-0.0115" mass="${link6_mass}" ixx="0.00006649"
+      iyy="0.00006649" izz="0.000096" />
     <visual>
       <geometry>
@@ -126,5 +141,5 @@
     </collision>
   </link>
-  <joint name="joint2_to_joint1" type="revolute">
+  <joint name="joint1" type="revolute">
     <axis xyz="0 0 1" />
     <limit effort="1000.0" lower="-2.93" upper="2.93" velocity="0" />
@@ -132,7 +147,7 @@
     <child link="link1" />
     <origin xyz="0 0 0.1739" rpy="0 0 0" />
-    <dynamics damping="${joint_damping}" friction="${joint_friction}"/>
-  </joint>
-  <joint name="joint3_to_joint2" type="revolute">
+    <dynamics damping="${joint_damping}" friction="${joint_friction}" />
+  </joint>
+  <joint name="joint2" type="revolute">
     <axis xyz="0 0 1" />
     <limit effort="1000.0" lower="-2.35" upper="2.35" velocity="0" />
@@ -140,7 +155,7 @@
     <child link="link2" />
     <origin xyz="0 -0.08878 0" rpy="0 -1.5708 1.5708" />
-    <dynamics damping="${joint_damping}" friction="${joint_friction}"/>
-  </joint>
-  <joint name="joint4_to_joint3" type="revolute">
+    <dynamics damping="${joint_damping}" friction="${joint_friction}" />
+  </joint>
+  <joint name="joint3" type="revolute">
     <axis xyz=" 0 0 1" />
     <limit effort="1000.0" lower="-2.53" upper="2.53" velocity="0" />
@@ -148,7 +163,7 @@
     <child link="link3" />
     <origin xyz="0.135 0 -0.08878   " rpy="0 0 0" />
-    <dynamics damping="${joint_damping}" friction="${joint_friction}"/>
-  </joint>
-  <joint name="joint5_to_joint4" type="revolute">
+    <dynamics damping="${joint_damping}" friction="${joint_friction}" />
+  </joint>
+  <joint name="joint4" type="revolute">
     <axis xyz=" 0 0 1" />
     <limit effort="1000.0" lower="-2.53" upper="2.53" velocity="0" />
@@ -156,7 +171,7 @@
     <child link="link4" />
     <origin xyz="0.120 0 0.08878 " rpy=" 0 0 1.57080" />
-    <dynamics damping="${joint_damping}" friction="${joint_friction}"/>
-  </joint>
-  <joint name="joint6_to_joint5" type="revolute">
+    <dynamics damping="${joint_damping}" friction="${joint_friction}" />
+  </joint>
+  <joint name="joint5" type="revolute">
     <axis xyz="0 0 1" />
     <limit effort="1000.0" lower="-2.93" upper="2.93" velocity="0" />
@@ -164,7 +179,7 @@
     <child link="link5" />
     <origin xyz="0 -0.095 0.0" rpy="1.5708 0 0" />
-    <dynamics damping="${joint_damping}" friction="${joint_friction}"/>
-  </joint>
-  <joint name="joint6output_to_joint6" type="revolute">
+    <dynamics damping="${joint_damping}" friction="${joint_friction}" />
+  </joint>
+  <joint name="joint6" type="revolute">
     <axis xyz="0 0 1" />
     <limit effort="1000.0" lower="-3.14" upper="3.14" velocity="0" />
@@ -172,5 +187,30 @@
     <child link="link6" />
     <origin xyz="0 0.0655 0.0" rpy="-1.5708 0 0" />
-    <dynamics damping="${joint_damping}" friction="${joint_friction}"/>
-  </joint>
+    <dynamics damping="${joint_damping}" friction="${joint_friction}" />
+  </joint>
+  <!-- CONFIGURACION DE PLUGINS DE GAZEBO  *******************-->
+  <xacro:macro name="apply_joint_force" params="joint">
+    <plugin filename="gz-sim-apply-joint-force-system"
+      name="gz::sim::systems::ApplyJointForce">
+      <joint_name>${joint}</joint_name>
+    </plugin>
+  </xacro:macro>
+  <gazebo>
+    <!-- Este plugin publica el estado de las articulaciones -->
+    <plugin filename="gz-sim-joint-state-publisher-system"
+      name="gz::sim::systems::JointStatePublisher">
+    </plugin>
+    <!-- Plugins para aplicar fuerzas/torques desde ROS2 a las juntas -->
+    <xacro:apply_joint_force joint="joint1" />
+    <xacro:apply_joint_force joint="joint2" />
+    <xacro:apply_joint_force joint="joint3" />
+    <xacro:apply_joint_force joint="joint4" />
+    <xacro:apply_joint_force joint="joint5" />
+    <xacro:apply_joint_force joint="joint6" />
+  </gazebo>
+  <!--  CONFIGURACION DE COLISIONES *******************-->
+  <!-- Self collision -->
+  <gazebo>
+    <self_collide>false</self_collide>
+  </gazebo>
 </robot>
